File: SegmentDriver/SegmentDriver.brd (EAGLE design)
At the start: 160 x 100 mm, 68 parts, among them K1 M02-MOLEX-104188-0210, K2 M02-MOLEX-104188-0210, K3 M02-MOLEX-104188-0210, K4 M02-MOLEX-104188-0210, K5 M02-MOLEX-104188-0210, K6 M02-MOLEX-104188-0210, K7 M02-MOLEX-104188-0210, K8 M02-MOLEX-104188-0210, K9 M02-MOLEX-104188-0210, Q1 MOSFET-NCHANNEL-FDMS5672, Q2 MOSFET-NCHANNEL-FDMS5672, Q3 MOSFET-NCHANNEL-FDMS5672, Q4 MOSFET-NCHANNEL-FDMS5672, Q5 MOSFET-NCHANNEL-FDMS5672, Q6 MOSFET-NCHANNEL-FDMS5672, Q7 MOSFET-NCHANNEL-FDMS5672, Q8 MOSFET-NCHANNEL-FDMS5672, Q9 MOSFET-NCHANNEL-FDMS5672, U1 FOD8321, U10 FOD8321, U13 DS1307SO8-TIGHT, U2 FOD8321, U3 FOD8321, U5 FOD8321, U6 FOD8321, U7 FOD8321, U8 FOD8321, U9 FOD8321, X1 32.768kHz

Commit message: Implemented RTD and RS485
Parts:
- removed K3, K5, K6, K7, K8, K9: M02-MOLEX-104188-0210, simbits:LITE-TRAP-CONNECTOR-2
- removed TP107: TEST-POINT3, SparkFun-Passives:PAD.03X.03
- added C11, C13, C15, C17, C18, C25: 47UF, Panasonic-EEEFK_EEEFP:CAPAE830X1050N
- added C12, C14, C16: 0.1uF, rcl:C1206K
- added C26, C27, C28, C29, C30, C33, C35, C36, C38, C39, C40, C41, C42, C43, C44, C45, C46, C47, C48, C49, C50, C51, C52, C53, C54, C55, C56, C57, C58, C59, C61, C62, C63, C64, C65, C66, C67, C68, C69, C70, C71, C73, C77, C78: 0.1uF, rcl:C0603K
- added C31, C32: 12pF, rcl:C0603K
- added C34, C37, C60: 1uF, rcl:C0603K
- added C72, C74, C75, C76: 220UF, Panasonic-EEEFK_EEEFP:CAPAE830X1050N
- added H1, H2, H3, H4: MOUNT-PAD-ROUND3.0, simbits:3,0-PAD
- added IC2: ATMEGA644A, atmel:TQFP44
- added K17: 61200621621, Wire-to-Board:61200621621
- added K18: 61201021621, Wire-to-Board:61201021621
- added KD1, KD2, KS1, KS2, KS3, KS4, KS5, KS6, KS7: M02-MOLEX-104188-0210, simbits:LITE-TRAP-CONNECTOR-2
- added KT1, KT2, KT3, KT4, KT5, KT6, KT7, KTD1, KTD2: 691321100004, Wurth_Elektronik_Electromechanic_Terminal_Blocks_Connectors_rev15d:691321100004
- added LED1, LED2: (no value), led:LED5MM
- added LED5, LED6: (no value), adafruit:CHIPLED_0603
- added LED7, LED8: AMBER, adafruit:CHIPLED_0603
- added Q10, Q11: (no value), simbits:SOT523
- added R18, R31, R35, R53, R54: 1k, rcl:R0603
- added R19, R20, R21, R22, R23, R24, R25, R26, R27, R29, R30, R34, R36: 0R, rcl:R0603
- added R28: 10k, rcl:R0603
- added R32, R33: 4.7k, rcl:R0603
- added R37, R38, R39, R40, R41, R42, R43, R44, R45, R46: 100k, rcl:R0603
- added R47: 1.2K, rcl:R0603
- added R48: 2K4, rcl:R0603
- added RESET_SW: SPST_TACT-EVQQ2, adafruit:EVQ-Q2
- added U14: (no value), simbits:TSSOP28
- added Y1: (no value), SparkFun-FreqCtrl:CRYSTAL-SMD-5X3
- C19, C20, C23: value 1uF -> 0.1uF
- C3, C4, C6: value 0.1uF -> 47UF; device rcl:C1206K -> Panasonic-EEEFK_EEEFP:CAPAE830X1050N
- K1, K2: value M02-MOLEX-104188-0210 -> 691318500002; device simbits:LITE-TRAP-CONNECTOR-2 -> TerminalBlocks:691318500002
- K4: value M02-MOLEX-104188-0210 -> 691321100005; device simbits:LITE-TRAP-CONNECTOR-2 -> Wurth_Elektronik_Electromechanic_Terminal_Blocks_Connectors_rev15d:691321100005
- R11: value 330R -> 100k
- R12: value 1K21 -> 100k
- R13: value 205R -> 0R
- R14, R16: value 330R -> 0R
- R15, R17: value 1K21 -> 0R
- U15: device simbits:TSSOP28 -> LINE_DRIVERS:SOIC08
- moved K2 936.0 mm to (-47.0, -825.0), turned to 0 degrees
- moved K1 914.7 mm to (-47.0, -801.0), turned to 0 degrees
- moved K4 845.4 mm to (-50.0, -736.0), turned to 0 degrees
- moved U15 782.3 mm to (-26.0, -753.0), turned to 0 degrees
- moved U2 246.2 mm to (-55.0, 207.0), turned to 90 degrees
- moved R2 227.6 mm to (-17.0, 211.0), turned to 90 degrees
- moved Q2 225.8 mm to (-39.0, 208.0)
- moved R7 222.8 mm to (243.0, 211.0), turned to 90 degrees
- moved C2 216.5 mm to (-16.0, 206.0)
- moved U3 200.8 mm to (-3.00, 207.0), turned to 90 degrees
- moved C24 198.9 mm to (232.0, 201.0)
- moved C23 193.6 mm to (226.0, 201.0)
- moved R3 190.6 mm to (35.0, 211.0), turned to 90 degrees
- moved R15 189.7 mm to (216.0, 201.0)
- moved R16 189.4 mm to (221.0, 201.0)
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Connections:
- removed net N$14 (its old number): K4.1A, K4.1B, Q4.D5, Q4.D6, Q4.D7, Q4.D8, Q4.DPAD
- removed net N$16 (its old number): K6.1A, K6.1B, Q6.D5, Q6.D6, Q6.D7, Q6.D8, Q6.DPAD
- removed net N$7 (its old number): K3.1A, K3.1B, Q3.D5, Q3.D6, Q3.D7, Q3.D8, Q3.DPAD
- removed net T5: C22.1, R11.2, R15.2
- removed net T6: C24.1, R16.2, R17.2
- removed net TREF: C20.1, R14.1
- new net !INT_PROJECTOR: IC2.12
- new net !RESET: IC2.4, K17.5, K18.6, R28.1, RESET_SW.A, RESET_SW.A'
- new net AD1_!CS: U11.24
- new net AD1_!DRDY: U11.25
- new net AD1_!RESET: R11.1, U11.4
- new net AD1_AIN0: KT1.4, U11.11
- new net AD1_AIN1: C19.2, C20.1, R13.1, U11.12
- new net AD1_AIN2: C19.1, C22.2, R14.1, U11.17
- new net AD1_AIN3: KT2.4, U11.18
- new net AD1_AIN4: C23.2, C24.1, R15.1, U11.13
- new net AD1_AIN5: C23.1, C38.2, R16.1, U11.14
- new net AD1_AIN6: C39.2, C40.1, R17.1, U11.15
- new net AD1_AIN7: C39.1, C41.2, R19.1, U11.16
- new net AD1_BIASP: KT1.1, KT2.1, KT3.1, R38.2, R39.1
- new net AD1_IEXC1: KT3.4
- new net AD1_START: U11.23
- new net AD2_!CS: U12.24
- new net AD2_!DRDY: U12.25
- new net AD2_!RESET: R12.1, U12.4
- new net AD2_AIN0: KT4.4, U12.11
- new net AD2_AIN1: C42.2, C43.1, R20.1, U12.12
- new net AD2_AIN2: C42.1, C44.2, R21.1, U12.17
- new net AD2_AIN3: KT5.4, U12.18
- new net AD2_AIN4: C45.2, C46.1, R22.1, U12.13
- new net AD2_AIN5: C45.1, C47.2, R23.1, U12.14
- new net AD2_AIN6: C48.2, C49.1, R24.1, U12.15
- new net AD2_AIN7: C48.1, C50.2, R25.1, U12.16
- new net AD2_BIASP: KT4.1, KT5.1, KT6.1, R41.2, R42.1, R44.2, R45.1
- new net AD2_IEXC1: KT6.4
- new net AD2_START: U12.23
- new net AD3_!CS: U14.24
- new net AD3_!DRDY: U14.25
- new net AD3_!RESET: R37.1, U14.4
- new net AD3_AIN0: KT7.4, U14.11
- new net AD3_AIN1: C51.2, C52.1, R26.1, U14.12
- new net AD3_AIN2: C51.1, C53.2, R27.1, U14.17
- new net AD3_AIN3: KTD1.4, U14.18
- new net AD3_AIN4: C54.2, C55.1, R29.1, U14.13
- new net AD3_AIN5: C54.1, C56.2, R30.1, U14.14
- new net AD3_AIN6: C57.2, C58.1, R34.1, U14.15
- new net AD3_AIN7: C57.1, C59.2, R36.1, U14.16
- new net AD3_BIASP: KT7.1, KTD1.1, KTD2.1
- new net AD3_IEXC1: KTD2.4
- new net AD3_START: U14.23
- new net AVDD: C33.1, C36.1, C62.1, U11.22, U12.22, U14.22
- new net CS_ADS1248_1: IC2.35
- new net CS_ADS1248_2: IC2.36
- new net CS_ADS1248_3: IC2.37
- new net DVDD: C21.1, C35.1, C61.1, R11.2, R12.2, R37.2, U11.1, U12.1, U14.1
- new net LED1: IC2.30, R35.1
- new net LED2: IC2.31, R31.1
- new net MISO: IC2.2, K17.1, U11.26, U12.26, U14.26
- new net MOSI: IC2.1, K17.4, U11.27, U12.27, U14.27
- new net N$11: C11.1, KS4.1A, KS4.1B, Q4.D5, Q4.D6, Q4.D7, Q4.D8, Q4.DPAD
- new net N$13: C13.1, KS5.1A, KS5.1B, Q5.D5, Q5.D6, Q5.D7, Q5.D8, Q5.DPAD
- new net N$25: LED7.C, R53.2
- new net N$26: LED8.C, R54.2
- new net N$27: KT1.2, R14.2
- new net N$28: KT3.3, R17.2
- new net N$29: C29.2, IC2.29
- new net N$30: C34.1, U11.9
- new net N$31: KT3.2, R19.2
- new net N$32: LED5.A, R31.2
- new net N$33: LED6.A, R35.2
- new net N$34: KT4.3, R20.2
- new net N$35: KT4.2, R21.2
- new net N$36: IC2.26
- new net N$37: IC2.25
- new net N$38: IC2.16
- new net N$39: C32.1, IC2.8, Y1.1
- new net N$40: C31.1, IC2.7, Y1.3
- new net N$41: C37.1, U12.9
- new net N$42: KT5.3, R22.2
- new net N$43: KT5.2, R23.2
- new net N$44: KT6.3, R24.2
- new net N$45: KT6.2, R25.2
- new net N$46: KT7.3, R26.2
- new net N$47: IC2.9, R18.2
- new net N$48: KT7.2, R27.2
- new net N$49: KTD1.3, R29.2
- new net N$50: KTD1.2, R30.2
- new net N$51: KTD2.3, R34.2
- new net N$52: KTD2.2, R36.2
- new net N$53: C60.1, U14.9
- new net N$54: C67.2, C68.1, R43.2, U12.6
- new net N$55: C64.2, C65.1, R40.2, U11.6
- new net N$56: C66.2, C67.1, R42.2, U12.5
- new net N$57: C63.2, C64.1, R39.2, U11.5
- new net N$58: C70.2, C71.1, R46.2, U14.6
- new net N$59: C69.2, C70.1, R45.2, U14.5
- new net N$60: Q11.3, R54.1
- new net N$61: Q10.3, R53.1
- new net N$62: LED2.A, R47.1
- new net N$63: LED1.A, R48.1
- new net N$64: U15.2
- new net N$8: C6.1, KS3.1A, KS3.1B, Q3.D5, Q3.D6, Q3.D7, Q3.D8, Q3.DPAD
- new net POWERFAIL: IC2.15
- new net POWERGOOD: IC2.14
- new net PWRON: IC2.13
- new net RS485+: K4.1, K4.3, U15.6
- new net RS485-: K4.2, K4.4, U15.7
- new net SCK: IC2.3, K17.3, U11.28, U12.28, U14.28
- new net TCK: IC2.21, K18.1
- new net TDI: IC2.24, K18.9
- new net TDO: IC2.23, K18.3
- new net TMS: IC2.22, K18.5
- new net UART_DE: IC2.32, U15.3
- new net UART_RX: Q10.1, R18.1, U15.1
- new net UART_TX: IC2.10, Q11.1, U15.4
- net +12V: now also C12.1, C14.1, C16.1, C74.1, C75.1, C77.2, K2.2, R47.2; no longer C3.1, C4.1, C6.1
- net +24V: now also C72.1, C76.1, C78.2, K1.2, KD1.2A, KD1.2B, KD2.2A, KD2.2B, KS1.2A, KS1.2B, KS2.2A, KS2.2B, KS3.2A, KS3.2B, KS4.2A, KS4.2B, KS5.2A, KS5.2B, KS6.2A, KS6.2B, KS7.2A, KS7.2B, R48.2; no longer K1.2A, K1.2B, K2.2A, K2.2B, K3.2A, K3.2B, K4.2A, K4.2B, K5.2A, K5.2B, K6.2A, K6.2B, K7.2A, K7.2B, K8.2A, K8.2B, K9.2A, K9.2B
- net 3.3V: now also C73.1, LED7.A, LED8.A, U15.8; no longer R12.1, R15.1, R17.1
- net 5V: now also C26.2, C27.2, C28.2, C30.2, IC2.17, IC2.27, IC2.38, IC2.5, K17.2, K18.4, R28.2, R32.2, R33.2
- net AGND: now also C11.2, C13.2, C15.2, C17.2, C18.2, C25.2, C3.2, C4.2, C6.2
- net GND: now also C12.2, C14.2, C16.2, C22.1, C26.1, C27.1, C28.1, C29.1, C30.1, C31.2, C32.2, C33.2, C34.2, C35.2, C36.2, C37.2, C38.1, C40.2, C41.1, C43.2, C44.1, C46.2, C47.1, C49.2, C50.1, C52.2, C53.1, C55.2, C56.1, C58.2, C59.1, C60.2, C61.2, C62.2, C63.1, C65.2, C66.1, C68.2, C69.1, C71.2, C72.2, C73.2, C74.2, C75.2, C76.2, C77.1, C78.1, H1.B3,0, H2.B3,0, H3.B3,0, H4.B3,0, IC2.18, IC2.28, IC2.39, IC2.6, K1.1, K17.6, K18.10, K18.2, K2.1, LED1.K, LED2.K, LED5.C, LED6.C, Q10.2, Q11.2, R38.1, R40.1, R41.1, R43.1, R44.1, R46.1, RESET_SW.B, RESET_SW.B', U11.10, U11.2, U11.21, U11.3, U12.10, U12.2, U12.21, U12.3, U14.10, U14.2, U14.21, U14.3, U15.5; no longer C19.2, C22.2, C23.2, C3.2, C4.2, C6.2, R13.2, U15.27
- net IIC1_SCL: now also IC2.19, R32.1
- net IIC1_SDA: now also IC2.20, R33.1
- net N$15: now also C15.1, KS6.1A, KS6.1B, Q6.D5, Q6.D6, Q6.D7, Q6.D8, Q6.DPAD; no longer K5.1A, K5.1B, Q5.D5, Q5.D6, Q5.D7, Q5.D8, Q5.DPAD
- net N$17: now also C17.1, KS7.1A, KS7.1B; no longer K7.1A, K7.1B
- net N$18: now also C18.1, KD1.1A, KD1.1B; no longer K9.1A, K9.1B
- net N$19: now also C25.1, KD2.1A, KD2.1B; no longer K8.1A, K8.1B
- net N$20: now also KT2.3, R15.2; no longer C19.1, R11.1
- net N$22: now also KT2.2, R16.2; no longer R12.2, R13.1, R14.2, TP107.P$1
- net N$23: now also KT1.3, R13.2; no longer C23.1, R16.1
- net N$3: now also C3.1, KS1.1A, KS1.1B; no longer K1.1A, K1.1B
- net N$6: now also C4.1, KS2.1A, KS2.1B; no longer K2.1A, K2.1B
- net PWM_DOT1: now also R9.1; no longer R8.1
- net PWM_DOT2: now also R8.1; no longer R9.1
- net RTC_1HZ_CLK: now also IC2.11
Other:
- board size 160 x 100 mm -> 200 x 200 mm

Commit message: Added ext. gpio, 7 seg. driver, differential filtering
Parts:
- removed K4: 691321100005, Wurth_Elektronik_Electromechanic_Terminal_Blocks_Connectors_rev15d:691321100005
- removed LED2: (no value), led:LED5MM
- added C79, C80: 0.1uF, rcl:C0603K
- added IC1: PCA9555PW, micro-philips:TSSOP24
- added IC3: 4511D, 45xx:SO16
- added K3: (no value), Wurth_Elektronik_Electromechanic_Input-Output_Connectors_rev15c:615016149521
- added KB1, KB2, KB3, KB4, KB5, KB6: 53261-03, con-molex:53261-03
- added R49, R50, R51, R52, R55, R69: 33R, simbits:RESCAV80P320X160X70-8N
- added R56, R57, R59: 47R, simbits:RESCAV80P320X160X70-8N
- added R58: 10k, rcl:R0603
- added R60: 1k, simbits:RESCAV80P320X160X70-8N
- C11, C13, C15, C17, C18, C25, C3, C4, C6: value 47UF -> 470UF; device Panasonic-EEEFK_EEEFP:CAPAE830X1050N -> Panasonic-EEEFK_EEEFP:CAPAE1700X1700N
- C72, C76: value 220UF -> 470UF; device Panasonic-EEEFK_EEEFP:CAPAE830X1050N -> Panasonic-EEEFK_EEEFP:CAPAE1700X1700N
- KT1, KT2, KT3, KT4, KT5, KT6, KT7, KTD1, KTD2: value 691321100004 -> 691210910004; device Wurth_Elektronik_Electromechanic_Terminal_Blocks_Connectors_rev15d:691321100004 -> Wurth_Elektronik_Electromechanic_Terminal_Blocks_Connectors_rev15d:691210910004
- LED1: value (none) -> 7-SEG_SA02-107; device led:LED5MM -> display-kingbright-2:SA02107
- Q10, Q11: value (none) -> DMP2215L-7; device simbits:SOT523 -> simbits:SOT95P240X110-3N
- moved C78 1015.0 mm to (2.00, 145.0)
- moved C76 962.8 mm to (20.0, 117.0)
- moved C72 958.1 mm to (20.0, 136.0)
- moved C77 939.3 mm to (47.0, 82.0)
- moved R47 939.3 mm to (36.0, 82.0)
- moved R48 939.3 mm to (42.0, 82.0)
- moved LED1 938.9 mm to (183.0, 49.0), turned to 180 degrees
- moved C75 931.5 mm to (16.0, 85.0)
- moved K1 929.5 mm to (5.00, 127.0), turned to 90 degrees
- moved C74 921.7 mm to (16.0, 74.0)
- moved K2 908.5 mm to (6.00, 82.0), turned to 90 degrees
- moved C73 828.0 mm to (150.0, 16.0)
- moved LED7 828.0 mm to (165.0, 29.0)
- moved LED8 828.0 mm to (170.0, 29.0)
- moved R53 828.0 mm to (172.0, 21.0)
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Connections:
- removed net !INT_PROJECTOR: IC2.12
- removed net 3.3V: C73.1, LED7.A, LED8.A, U15.8
- removed net POWERFAIL: IC2.15
- removed net POWERGOOD: IC2.14
- removed net PWRON: IC2.13
- new net EXTGPIO_!INT: IC1.1, IC2.12, R58.1
- new net GPIO1: KB1.2, R56.8
- new net GPIO2: KB2.2, R56.7
- new net GPIO3: KB3.2, R56.6
- new net GPIO4: KB4.2, R56.5
- new net GPIO5: KB5.2, R57.8
- new net GPIO6: KB6.2, R57.7
- new net GPIO7: R57.6
- new net GPIO8: R57.5
- new net N$100: LED1.E@1, R60.8
- new net N$101: LED1.F@9, R60.7
- new net N$102: LED1.G@10, R60.6
- new net N$103: LED1.DP@5, R60.5
- new net N$104: IC1.14, IC3.1
- new net N$105: IC1.15, IC3.2
- new net N$106: IC1.16, IC3.6
- new net N$107: IC1.17, IC3.5
- new net N$108: IC1.18, R60.4
- new net N$65: R49.5, U11.25
- new net N$66: R69.8, U11.24
- new net N$67: R69.7, U11.27
- new net N$68: R69.6, U11.26
- new net N$69: R69.5, U11.28
- new net N$70: R49.8, U11.23
- new net N$71: R51.5, U14.28
- new net N$72: R51.6, U14.26
- new net N$73: R51.7, U14.27
- new net N$74: R51.8, U14.24
- new net N$75: R50.5, U14.25
- new net N$76: R50.8, U14.23
- new net N$77: R52.5, U12.28
- new net N$78: R52.6, U12.26
- new net N$79: R52.7, U12.27
- new net N$80: R52.8, U12.24
- new net N$81: R55.5, U12.25
- new net N$82: R55.8, U12.23
- new net N$83: IC1.7, R56.4
- new net N$84: IC1.8, R57.1
- new net N$85: IC1.9, R57.2
- new net N$86: IC1.10, R57.3
- new net N$87: IC1.11, R57.4
- new net N$88: IC1.13, IC3.7
- new net N$89: IC3.13, R59.1
- new net N$90: IC3.12, R59.2
- new net N$91: IC3.11, R59.3
- new net N$92: IC3.10, R59.4
- new net N$93: IC3.9, R60.1
- new net N$94: IC3.15, R60.2
- new net N$95: IC3.14, R60.3
- new net N$96: LED1.A@7, R59.8
- new net N$97: LED1.B@6, R59.7
- new net N$98: LED1.C@4, R59.6
- new net N$99: LED1.D@2, R59.5
- net +5V: now also C73.1, C79.1, C80.1, IC1.24, IC3.16, IC3.3, IC3.4, KB1.1, KB2.1, KB3.1, KB4.1, KB5.1, KB6.1, Q10.2, Q11.2, R58.2, U15.8
- net AD1_!CS: now also R69.1; no longer U11.24
- net AD1_!DRDY: now also R49.4; no longer U11.25
- net AD1_START: now also R49.1; no longer U11.23
- net AD2_!CS: now also R52.1; no longer U12.24
- net AD2_!DRDY: now also R55.4; no longer U12.25
- net AD2_START: now also R55.1; no longer U12.23
- net AD3_!CS: now also R51.1; no longer U14.24
- net AD3_!DRDY: now also R50.4; no longer U14.25
- net AD3_START: now also R50.1; no longer U14.23
- net GND: now also C79.2, C80.2, IC1.12, IC1.2, IC1.21, IC1.3, IC3.8, KB1.3, KB2.3, KB3.3, KB4.3, KB5.3, KB6.3, LED1.COM@3, LED1.COM@8, R53.1, R54.1; no longer LED1.K, LED2.K, Q10.2, Q11.2
- net IIC1_SCL: now also IC1.22
- net IIC1_SDA: now also IC1.23
- net MISO: now also R51.3, R52.3, R69.3; no longer U11.26, U12.26, U14.26
- net MOSI: now also R51.2, R52.2, R69.2; no longer U11.27, U12.27, U14.27
- net N$36: now also IC1.4, R56.1; no longer IC2.26
- net N$37: now also IC1.5, R56.2; no longer IC2.25
- net N$38: now also IC1.6, R56.3; no longer IC2.16
- net N$60: now also LED7.A, Q10.3; no longer Q11.3, R54.1
- net N$61: now also LED8.A, Q11.3; no longer Q10.3, R53.1
- net N$62: no longer LED2.A
- net N$63: no longer LED1.A
- net RS485+: now also K3.A2, K3.B1; no longer K4.1, K4.3
- net RS485-: now also K3.A1, K3.B2; no longer K4.2, K4.4
- net SCK: now also R51.4, R52.4, R69.4; no longer U11.28, U12.28, U14.28

Commit message: reduced size to 175mm
Parts:
- added H5, H6, H7, H8: MOUNT-HOLE2.0, simbits:2,0
- added H9: MOUNT-PAD-ROUND2,0, simbits:2,0-PAD
- added K4: 691313710002, Wurth_Elektronik_Electromechanic_Terminal_Blocks_Connectors_rev15d:691313710002
- added K5: 691322310002, Wurth_Elektronik_Electromechanic_Terminal_Blocks_Connectors_rev15d:691322310002
- added LED2, LED3: (no value), adafruit:CHIPLED_0603
- C11, C13, C15, C17, C18, C25, C3, C4, C6: value 470UF -> 220UF; device Panasonic-EEEFK_EEEFP:CAPAE1700X1700N -> Panasonic-EEEFK_EEEFP:CAPAE1350X1400N
- H1, H2, H3, H4: value MOUNT-PAD-ROUND3.0 -> MOUNT-PAD-ROUND2,0; device simbits:3,0-PAD -> simbits:2,0-PAD
- K1: value 691318500002 -> 691313710002; device TerminalBlocks:691318500002 -> Wurth_Elektronik_Electromechanic_Terminal_Blocks_Connectors_rev15d:691313710002
- K2: value 691318500002 -> 691322310002; device TerminalBlocks:691318500002 -> Wurth_Elektronik_Electromechanic_Terminal_Blocks_Connectors_rev15d:691322310002
- moved C80 248.4 mm to (186.0, 26.0)
- moved IC3 248.4 mm to (191.0, 35.0)
- moved R7 198.7 mm to (72.0, 92.0), turned to 90 degrees
- moved R4 188.2 mm to (93.0, 92.0)
- moved Q7 183.2 mm to (51.5, 127.5), turned to 90 degrees
- moved U8 170.4 mm to (73.5, 101.0), turned to 0 degrees
- moved C16 165.2 mm to (108.5, 109.5), turned to 0 degrees
- moved U5 163.6 mm to (94.5, 101.0), turned to 0 degrees
- moved R6 159.8 mm to (79.0, 92.0), turned to 90 degrees
- moved C7 156.7 mm to (116.0, 109.5), turned to 0 degrees
- moved R3 153.4 mm to (99.5, 92.0), turned to 90 degrees
- moved C5 152.9 mm to (94.5, 109.5), turned to 0 degrees
- moved Q6 148.1 mm to (69.5, 127.5), turned to 90 degrees
- moved Q4 146.6 mm to (105.5, 127.5), turned to 90 degrees
- moved C12 144.1 mm to (73.5, 109.5), turned to 0 degrees
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Connections:
- net +12V: now also K2.1, K5.2; no longer K2.2
- net +24V: now also K1.1, K4.2; no longer K1.2
- net GND: now also H1.B2,2, H2.B2,2, H3.B2,2, H4.B2,2, H9.B2,2, K1.2, K2.2, K4.1, K5.1, LED2.C, LED3.C; no longer H1.B3,0, H2.B3,0, H3.B3,0, H4.B3,0, K1.1, K2.1
- net N$62: now also LED3.A
- net N$63: now also LED2.A
Routing:
- net VO: track 0.00 -> 58.2 mm
- net VO8: track 0.00 -> 54.1 mm
- net VO1: track 0.00 -> 48.2 mm
- net VO7: track 0.00 -> 44.2 mm
- net VO2: track 0.00 -> 37.2 mm
- net VO6: track 0.00 -> 34.4 mm
- net +12V: track 0.00 -> 30.6 mm
- net GND: track 0.00 -> 29.2 mm
- net VO3: track 0.00 -> 28.6 mm
- net VO5: track 0.00 -> 22.2 mm
- net VO4: track 0.00 -> 19.3 mm
Other:
- board size 200 x 200 mm -> 174.5 x 175 mm

Commit message: routing rtd inputs
Parts:
- removed H9: MOUNT-PAD-ROUND2,0, simbits:2,0-PAD
- removed KB1: 53261-03, con-molex:53261-03
- removed KT1, KT2: 691210910004, Wurth_Elektronik_Electromechanic_Terminal_Blocks_Connectors_rev15d:691210910004
- removed LED8: AMBER, adafruit:CHIPLED_0603
- removed Q10, Q11: DMP2215L-7, simbits:SOT95P240X110-3N
- removed R69: 33R, simbits:RESCAV80P320X160X70-8N
- added $2_206_$_2016-11-07_20-18-07: MOUNT-HOLE2.0, simbits:2,0
- added K6: 61200621621, Wire-to-Board:61200621621
- added K7: 61201021621, Wire-to-Board:61201021621
- added LED4: (no value), adafruit:CHIPLED_0603
- added R61: 1k, simbits:RESCAV80P320X160X70-8N
- added U16: DMP2215L-7, simbits:SOT95P240X110-3N
- added U17: (no value), LINE_DRIVERS:SOIC08
- added Y2: 32.768kHz, SparkFun-FreqCtrl:CRYSTAL-32KHZ-SMD_EPSON_MC146
- C1: value 0.1uF -> 470UF; device rcl:C1206K -> Panasonic-EEEFK_EEEFP:CAPAE1700X1700N
- C11: value 220UF -> 12pF; device Panasonic-EEEFK_EEEFP:CAPAE1350X1400N -> rcl:C0603K
- C12: value 0.1uF -> 12pF; device rcl:C1206K -> rcl:C0603K
- C13, C6: value 220UF -> 0.1uF; device Panasonic-EEEFK_EEEFP:CAPAE1350X1400N -> rcl:C0603K
- C14, C5, C7, C8, C9: device rcl:C1206K -> rcl:C0603K
- C15, C17, C18: value 220UF -> 0.1uF; device Panasonic-EEEFK_EEEFP:CAPAE1350X1400N -> rcl:C1206K
- C19, C20, C21, C22, C23: device rcl:C0603K -> rcl:C1206K
- C2: value 0.1uF -> 220UF; device rcl:C1206K -> Panasonic-EEEFK_EEEFP:CAPAE830X1050N
- C24, C26, C27, C28, C29, C30: value 0.1uF -> 220UF; device rcl:C0603K -> Panasonic-EEEFK_EEEFP:CAPAE1350X1400N
- C3: value 220UF -> 470UF; device Panasonic-EEEFK_EEEFP:CAPAE1350X1400N -> Panasonic-EEEFK_EEEFP:CAPAE1700X1700N
- C31, C32: value 12pF -> 220UF; device rcl:C0603K -> Panasonic-EEEFK_EEEFP:CAPAE1350X1400N
- C34, C37, C60: value 1uF -> 0.1uF
- C39, C40, C41: value 0.1uF -> 1uF
- C4: device Panasonic-EEEFK_EEEFP:CAPAE1350X1400N -> Panasonic-EEEFK_EEEFP:CAPAE830X1050N
- C72, C76: value 470UF -> 0.1uF; device Panasonic-EEEFK_EEEFP:CAPAE1700X1700N -> rcl:C0603K
- C74, C75: value 220UF -> 0.1uF; device Panasonic-EEEFK_EEEFP:CAPAE830X1050N -> rcl:C0603K
- H5: value MOUNT-HOLE2.0 -> MOUNT-PAD-ROUND2,0; device simbits:2,0 -> simbits:2,0-PAD
- IC1: value PCA9555PW -> ATMEGA644A; device micro-philips:TSSOP24 -> atmel:TQFP44
- IC2: value ATMEGA644A -> PCA9555PW; device atmel:TQFP44 -> micro-philips:TSSOP24
- K17: value 61200621621 -> 691210910004; device Wire-to-Board:61200621621 -> Wurth_Elektronik_Electromechanic_Terminal_Blocks_Connectors_rev15d:691210910004
- K18: value 61201021621 -> 691210910004; device Wire-to-Board:61201021621 -> Wurth_Elektronik_Electromechanic_Terminal_Blocks_Connectors_rev15d:691210910004
- K2: value 691322310002 -> 691313710002; device Wurth_Elektronik_Electromechanic_Terminal_Blocks_Connectors_rev15d:691322310002 -> Wurth_Elektronik_Electromechanic_Terminal_Blocks_Connectors_rev15d:691313710002
- K3: value (none) -> 691322310002; device Wurth_Elektronik_Electromechanic_Input-Output_Connectors_rev15c:615016149521 -> Wurth_Elektronik_Electromechanic_Terminal_Blocks_Connectors_rev15d:691322310002
- K4: value 691313710002 -> 691322310002; device Wurth_Elektronik_Electromechanic_Terminal_Blocks_Connectors_rev15d:691313710002 -> Wurth_Elektronik_Electromechanic_Terminal_Blocks_Connectors_rev15d:691322310002
- K5: value 691322310002 -> (none); device Wurth_Elektronik_Electromechanic_Terminal_Blocks_Connectors_rev15d:691322310002 -> Wurth_Elektronik_Electromechanic_Input-Output_Connectors_rev15c:615016149521
- LED1: value 7-SEG_SA02-107 -> (none); device display-kingbright-2:SA02107 -> adafruit:CHIPLED_0603
- LED5, LED6: value (none) -> AMBER
- LED7: value AMBER -> 7-SEG_SA02-107; device adafruit:CHIPLED_0603 -> display-kingbright-2:SA02107
- R1: value 330 -> 2K4
- R10: value 10k -> 330
- R11, R12: value 100k -> 330
- R13, R14, R15, R16, R17: value 0R -> 330
- R18: value 1k -> 330
- R19, R20, R21, R29, R30, R34, R36: value 0R -> 100k
- R2: value 330 -> 1.2K
- R22, R23, R24, R25, R26, R27: value 0R -> 33R; device rcl:R0603 -> simbits:RESCAV80P320X160X70-8N
- R28: value 10k -> 100k
- R3, R9: value 330 -> 10k
- R31, R35: value 1k -> 100k
- R32, R33: value 4.7k -> 100k
- R37, R38, R39, R40, R41, R42, R43, R44, R45, R46: value 100k -> 0R
- R4, R7, R8: value 330 -> 1k
- R47: value 1.2K -> 0R
- R48: value 2K4 -> 0R
- R49, R50, R51, R52: value 33R -> 0R; device simbits:RESCAV80P320X160X70-8N -> rcl:R0603
- R5, R6: value 330 -> 4.7k
- R53, R54: value 1k -> 0R
- R55: value 33R -> 1k; device simbits:RESCAV80P320X160X70-8N -> rcl:R0603
- R56: value 47R -> 1k; device simbits:RESCAV80P320X160X70-8N -> rcl:R0603
- R57: value 47R -> 10k; device simbits:RESCAV80P320X160X70-8N -> rcl:R0603
- R58: value 10k -> 47R; device rcl:R0603 -> simbits:RESCAV80P320X160X70-8N
- R60: value 1k -> 47R
- U1: value FOD8321 -> DS1307SO8-TIGHT; device simbits:WB-SOP5 -> SparkFun-FreqCtrl:SO08-TIGHT
- U11: value (none) -> FOD8321; device simbits:TSSOP28 -> simbits:WB-SOP5
- U13: value DS1307SO8-TIGHT -> (none); device SparkFun-FreqCtrl:SO08-TIGHT -> simbits:TSSOP28
- U15: value (none) -> DMP2215L-7; device LINE_DRIVERS:SOIC08 -> simbits:SOT95P240X110-3N
- U2: value FOD8321 -> (none); device simbits:WB-SOP5 -> adafruit:TSSOP28
- U4: value (none) -> FOD8321; device adafruit:TSSOP28 -> simbits:WB-SOP5
- X1: value 32.768kHz -> 53261-03; device SparkFun-FreqCtrl:CRYSTAL-32KHZ-SMD_EPSON_MC146 -> con-molex:53261-03
- moved C24 229.8 mm to (159.5, 147.5), turned to 270 degrees
- moved K3 229.1 mm to (8.00, 80.0), turned to 90 degrees
- moved BAT1 228.1 mm to (214.0, 96.6)
- moved C79 228.1 mm to (200.5, 69.5)
- moved LED2 221.9 mm to (191.5, 70.0)
- moved H5 186.7 mm to (4.00, 87.5)
- moved LED6 182.8 mm to (170.0, 29.0), turned to 0 degrees
- moved C78 173.6 mm to (150.0, 16.0)
- moved R34 170.1 mm to (11.2, 21.5), turned to 90 degrees
- moved LED5 167.3 mm to (165.0, 29.0), turned to 0 degrees
- moved C57 164.6 mm to (10.0, 9.00), turned to 90 degrees
- moved R38 159.4 mm to (11.5, 9.00), turned to 270 degrees
- moved R40 158.5 mm to (22.5, 9.00), turned to 270 degrees
- moved K2 157.8 mm to (164.5, 100.0)
- moved R44 156.6 mm to (44.5, 9.00), turned to 270 degrees
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- renumbered KB2 to X2, KB3 to X3, KB4 to X4, KB5 to X5, KB6 to X6, KD1 to K15, KD2 to K16, KS1 to K8, KS2 to K9, KS3 to K10, KS4 to K11, KS5 to K12, KS6 to K13, KS7 to K14, KT3 to K19, KT4 to K20, KT5 to K21, KT6 to K22, KT7 to K23, KTD1 to K24, KTD2 to K25, RESET_SW to SW1
Connections:
- removed net N$77: R52.5, U12.28
- removed net N$78: R52.6, U12.26
- removed net N$79: R52.7, U12.27
- removed net N$80: R52.8, U12.24
- removed net N$81: R55.5, U12.25
- removed net N$82: R55.8, U12.23
- new net AD1_REFN0: C43.2, C44.1, R29.2, U12.6
- new net AD1_REFP0: C42.2, C43.1, R28.2, U12.5
- new net AD2_REFN0: C46.2, C47.1, R31.2, U13.6
- new net AD2_REFP0: C45.2, C46.1, R30.2, U13.5
- new net AD3_REFN0: C49.2, C50.1, R33.2, U14.6
- new net AD3_REFP0: C48.2, C49.1, R32.2, U14.5
- net !RESET: now also IC1.4, K6.5, K7.6, R3.1; no longer IC2.4, K17.5, K18.6, R28.1
- net +12V: now also C15.1, C17.1, C18.1, C19.1, C20.1, C21.1, C22.1, C23.1, C4.1, C6.2, K3.1, K4.2, R2.2, U11.6, U4.6; no longer C1.1, C12.1, C14.1, C5.1, C7.1, C74.1, C75.1, C77.2, C8.1, C9.1, K2.1, K5.2, R47.2, U1.6, U2.6
- net +24V: now also C1.1, C3.1, C5.2, K2.2, R1.2; no longer C72.1, C76.1, C78.2, K4.2, R48.2
- net +5V: now also C14.1, C78.1, IC2.24, R57.2, R9.2, U15.2, U16.2, U17.8, U2.28, X1.1; no longer C10.1, C73.1, IC1.24, KB1.1, Q10.2, Q11.2, R10.2, R58.2, U15.8, U4.28
- net 5V: now also C10.2, C7.2, C8.2, C9.2, IC1.17, IC1.27, IC1.38, IC1.5, K6.2, K7.4, R3.2, R5.2, R6.2, U1.8; no longer C26.2, C27.2, C28.2, C30.2, IC2.17, IC2.27, IC2.38, IC2.5, K17.2, K18.4, R28.2, R32.2, R33.2, U13.8
- net AD1_!CS: now also R22.2; no longer R69.1
- net AD1_!DRDY: now also R22.3; no longer R49.4
- net AD1_!RESET: now also R19.1, U12.4; no longer R11.1, U11.4
- net AD1_AIN0: now also K17.4, U12.11; no longer KT1.4, U11.11
- net AD1_AIN1: now also C51.2, C54.1, R37.1, U12.12; no longer C19.2, C20.1, R13.1, U11.12
- net AD1_AIN2: now also C51.1, C57.2, R38.1, U12.17; no longer C19.1, C22.2, R14.1, U11.17
- net AD1_AIN3: now also K18.4, U12.18; no longer KT2.4, U11.18
- net AD1_AIN4: now also C52.2, C55.1, R39.1, U12.13; no longer C23.2, C24.1, R15.1, U11.13
- net AD1_AIN5: now also C52.1, C58.2, R40.1, U12.14; no longer C23.1, C38.2, R16.1, U11.14
- net AD1_AIN6: now also C53.2, C56.1, R41.1, U12.15; no longer C39.2, C40.1, R17.1, U11.15
- net AD1_AIN7: now also C53.1, C59.2, R42.1, U12.16; no longer C39.1, C41.2, R19.1, U11.16
- net AD1_BIASP: now also K17.1, K18.1, R28.1, R34.2; no longer KT1.1, KT2.1, R38.2, R39.1
- net AD1_IEXC1: now also U12.20
- net AD1_START: now also R22.1; no longer R49.1
- net AD2_!CS: now also R24.2; no longer R52.1
- net AD2_!DRDY: now also R24.3; no longer R55.4
- net AD2_!RESET: now also R20.1, U13.4; no longer R12.1, U12.4
- net AD2_AIN0: now also U13.11; no longer U12.11
- net AD2_AIN1: now also C60.2, C63.1, R43.1, U13.12; no longer C42.2, C43.1, R20.1, U12.12
- net AD2_AIN2: now also C60.1, C66.2, R44.1, U13.17; no longer C42.1, C44.2, R21.1, U12.17
- net AD2_AIN3: now also U13.18; no longer U12.18
- net AD2_AIN4: now also C61.2, C64.1, R45.1, U13.13; no longer C45.2, C46.1, R22.1, U12.13
- net AD2_AIN5: now also C61.1, C67.2, R46.1, U13.14; no longer C45.1, C47.2, R23.1, U12.14
- net AD2_AIN6: now also C62.2, C65.1, R47.1, U13.15; no longer C48.2, C49.1, R24.1, U12.15
- net AD2_AIN7: now also C62.1, C68.2, R48.1, U13.16; no longer C48.1, C50.2, R25.1, U12.16
- net AD2_BIASP: now also R30.1, R32.1, R35.2, R36.2; no longer R41.2, R42.1, R44.2, R45.1
- net AD2_IEXC1: now also U13.20
- net AD2_START: now also R24.1; no longer R55.1
- net AD3_!CS: now also R26.2; no longer R51.1
- net AD3_!DRDY: now also R26.3; no longer R50.4
- net AD3_!RESET: now also R21.1; no longer R37.1
- net AD3_AIN1: now also C69.2, C72.1, R49.1; no longer C51.2, C52.1, R26.1
- net AD3_AIN2: now also C69.1, C75.2, R50.1; no longer C51.1, C53.2, R27.1
- net AD3_AIN4: now also C70.2, C73.1, R51.1; no longer C54.2, C55.1, R29.1
- net AD3_AIN5: now also C70.1, C76.2, R52.1; no longer C54.1, C56.2, R30.1
- net AD3_AIN6: now also C71.2, C74.1, R53.1; no longer C57.2, C58.1, R34.1
- net AD3_AIN7: now also C71.1, C77.2, R54.1; no longer C57.1, C59.2, R36.1
- net AD3_IEXC1: now also U14.20
- net AD3_START: now also R26.1; no longer R50.1
- net AGND: now also C24.2, C26.2, C27.2, C28.2, C29.2, C30.2, C31.2, C32.2; no longer C11.2, C13.2, C15.2, C17.2, C18.2, C3.2, C4.2, C6.2
- net AVDD: now also C37.1, C38.1, U13.22; no longer C33.1, C62.1, U11.22
- net CS_ADS1248_1: now also IC1.35; no longer IC2.35
- net CS_ADS1248_2: now also IC1.36; no longer IC2.36
- net CS_ADS1248_3: now also IC1.37; no longer IC2.37
- net DVDD: now also C33.1, C34.1, R19.2, R20.2, R21.2, U13.1; no longer C21.1, C61.1, R11.2, R12.2, R37.2, U11.1
- net EXTGPIO_!INT: now also IC1.12, IC2.1, R57.1; no longer IC1.1, IC2.12, R58.1
- net GND: now also C10.1, C11.2, C13.1, C15.2, C17.2, C18.2, C19.2, C22.2, C23.2, C3.2, C38.2, C39.2, C4.2, C41.2, C42.1, C44.2, C45.1, C47.2, C48.1, C5.1, C50.2, C54.2, C56.2, C57.1, C58.1, C6.1, C63.2, C64.2, C67.1, C68.1, C7.1, C75.1, C76.1, C78.2, C8.1, C9.1, H5.B2,2, IC1.18, IC1.28, IC1.39, IC1.6, IC2.12, IC2.2, IC2.21, IC2.3, K2.1, K3.2, K6.6, K7.10, K7.2, LED1.C, LED4.C, LED7.COM@3, LED7.COM@8, R29.1, R31.1, R33.1, R34.1, R35.1, R36.1, R55.1, R56.1, U11.4, U13.10, U13.2, U13.21, U13.3, U17.5, U2.1, U2.14, U2.2, U2.24, U2.25, U2.5, X1.3; no longer C10.2, C22.1, C24.2, C26.1, C27.1, C28.1, C29.1, C30.1, C31.2, C32.2, C38.1, C41.1, C43.2, C44.1, C46.2, C47.1, C49.2, C5.2, C50.1, C52.2, C53.1, C56.1, C58.2, C60.2, C61.2, C62.2, C63.1, C68.2, C69.1, C7.2, C71.2, C75.2, C76.2, C78.1, C8.2, C9.2, H9.B2,2, IC1.12, IC1.2, IC1.21, IC1.3, IC2.18, IC2.28, IC2.39, IC2.6, K17.6, K18.10, K18.2, K2.2, K5.1, KB1.3, LED1.COM@3, LED1.COM@8, LED5.C, LED6.C, R38.1, R40.1, R41.1, R43.1, R44.1, R46.1, R53.1, R54.1, U1.3, U11.10, U11.2, U11.21, U13.4, U15.5, U4.1, U4.14, U4.2, U4.24, U4.25, U4.5
- net GPIO1: now also R58.8, X1.2; no longer KB1.2, R56.8
- net GPIO2: now also R58.7; no longer R56.7
- net GPIO3: now also R58.6; no longer R56.6
- net GPIO4: now also R58.5; no longer R56.5
- net GPIO5: now also R59.8; no longer R57.8
- net GPIO6: now also R59.7; no longer R57.7
- net GPIO7: now also R59.6; no longer R57.6
- net GPIO8: now also R59.5; no longer R57.5
- net IIC1_SCL: now also IC1.19, IC2.22, R5.1, U1.6, U2.26; no longer IC1.22, IC2.19, R32.1, U13.6, U4.26
- net IIC1_SDA: now also IC1.20, IC2.23, R6.1, U1.5, U2.27; no longer IC1.23, IC2.20, R33.1, U13.5, U4.27
- net LED1: now also IC1.30, R7.1; no longer IC2.30, R35.1
- net LED2: now also IC1.31, R8.1; no longer IC2.31, R31.1
- net MISO: now also IC1.2, K6.1, R22.4, R24.4, R26.4; no longer IC2.2, K17.1, R51.3, R52.3, R69.3
- net MOSI: now also IC1.1, K6.4, R23.1, R25.1, R27.1; no longer IC2.1, K17.4, R51.2, R52.2, R69.2
- net N$1: now also R18.2, U11.1; no longer R8.2, U9.1
- net N$10: now also R10.2, U3.1; no longer R1.2, U1.1
- net N$100: now also LED7.E@1, R61.8; no longer LED1.E@1, R60.8
- net N$101: now also LED7.F@9, R61.7; no longer LED1.F@9, R60.7
- net N$102: now also LED7.G@10, R61.6; no longer LED1.G@10, R60.6
- net N$103: now also LED7.DP@5, R61.5; no longer LED1.DP@5, R60.5
- net N$104: now also IC2.14; no longer IC1.14
- net N$105: now also IC2.15; no longer IC1.15
- net N$106: now also IC2.16; no longer IC1.16
- net N$107: now also IC2.17; no longer IC1.17
- net N$108: now also IC2.18, R61.4; no longer IC1.18, R60.4
- net N$11: now also C27.1; no longer C11.1
- net N$12: now also R14.2, U7.1; no longer R5.2, U6.1
- net N$13: now also C28.1; no longer C13.1
- net N$14: now also R15.2, U8.1; no longer R6.2, U7.1
- net N$15: now also C29.1; no longer C15.1
- net N$16: now also R16.2, U9.1; no longer R7.2, U8.1
- net N$17: now also C30.1; no longer C17.1
- net N$18: now also C31.1, Q8.D5, Q8.D6, Q8.D7, Q8.D8, Q8.DPAD; no longer C18.1, Q9.D5, Q9.D6, Q9.D7, Q9.D8, Q9.DPAD
- net N$19: now also C32.1, Q9.D5, Q9.D6, Q9.D7, Q9.D8, Q9.DPAD; no longer C25.1, Q8.D5, Q8.D6, Q8.D7, Q8.D8, Q8.DPAD
- net N$2: now also R17.2; no longer R9.2
- net N$20: now also K18.3, R39.2; no longer KT2.3, R15.2
- net N$21: now also U1.2, Y2.P$2; no longer U13.2, X1.P$2
- net N$22: now also K18.2, R40.2; no longer KT2.2, R16.2
- net N$23: now also K17.3, R37.2; no longer KT1.3, R13.2
- net N$24: now also U1.3; no longer U13.3
- net N$25: now also LED5.C, R55.2; no longer LED7.C, R53.2
- net N$26: now also LED6.C, R56.2; no longer LED8.C, R54.2
- net N$27: now also K17.2, R38.2; no longer KT1.2, R14.2
- net N$28: now also R41.2; no longer R17.2
- net N$29: now also C13.2, IC1.29; no longer C29.2, IC2.29
- net N$3: now also C24.1; no longer C3.1
- net N$30: now also C39.1, U12.9; no longer C34.1, U11.9
- net N$31: now also R42.2; no longer R19.2
- net N$32: now also LED4.A, R8.2; no longer LED5.A, R31.2
- net N$33: now also LED3.A, R7.2; no longer LED6.A, R35.2
- net N$34: now also R43.2; no longer R20.2
- net N$35: now also R44.2; no longer R21.2
- net N$36: now also IC2.4, R58.1; no longer IC1.4, R56.1
- net N$37: now also IC2.5, R58.2; no longer IC1.5, R56.2
- net N$38: now also IC2.6, R58.3; no longer IC1.6, R56.3
- net N$39: now also C12.1, IC1.8; no longer C32.1, IC2.8
- net N$4: now also R11.2, U4.1; no longer R2.2, U2.1
- net N$40: now also C11.1, IC1.7; no longer C31.1, IC2.7
- net N$41: now also C40.1, U13.9; no longer C37.1, U12.9
- net N$42: now also R45.2; no longer R22.2
- net N$43: now also R46.2; no longer R23.2
- net N$44: now also R47.2; no longer R24.2
- net N$45: now also R48.2; no longer R25.2
- net N$46: now also R49.2; no longer R26.2
- net N$47: now also IC1.9, R4.2; no longer IC2.9, R18.2
- net N$48: now also R50.2; no longer R27.2
- net N$49: now also R51.2; no longer R29.2
- net N$5: now also R9.1, U2.23; no longer R10.1, U4.23
- net N$50: now also R52.2; no longer R30.2
- net N$51: now also R53.2; no longer R34.2
- net N$52: now also R54.2; no longer R36.2
- net N$53: now also C41.1; no longer C60.1
- net N$54: now also R23.7, U12.28; no longer C67.2, C68.1, R43.2, U12.6
- net N$55: now also R23.8, U12.27; no longer C64.2, C65.1, R40.2, U11.6
- net N$56: now also R22.5, U12.26; no longer C66.2, C67.1, R42.2, U12.5
- net N$57: now also R22.6, U12.25; no longer C63.2, C64.1, R39.2, U11.5
- net N$58: now also R22.7, U12.24; no longer C70.2, C71.1, R46.2, U14.6
- net N$59: now also R22.8, U12.23; no longer C69.2, C70.1, R45.2, U14.5
- net N$6: now also C25.1; no longer C4.1
- net N$60: now also LED5.A, U15.3; no longer LED7.A, Q10.3
- net N$61: now also LED6.A, U16.3; no longer LED8.A, Q11.3
- net N$62: now also LED2.A, R2.1; no longer LED3.A, R47.1
- net N$63: now also LED1.A, R1.1; no longer LED2.A, R48.1
- net N$64: now also U17.2; no longer U15.2
- net N$65: now also R24.8, U13.23; no longer R49.5, U11.25
- net N$66: now also R24.6, U13.25; no longer R69.8, U11.24
- net N$67: now also R24.7, U13.24; no longer R69.7, U11.27
- net N$68: now also R25.8, U13.27; no longer R69.6, U11.26
- net N$69: now also R24.5, U13.26; no longer R69.5, U11.28
- net N$7: now also R12.2, U5.1; no longer R3.2, U3.1
- net N$70: now also R25.7, U13.28; no longer R49.8, U11.23
- net N$71: now also R26.8, U14.23; no longer R51.5, U14.28
- net N$72: now also R26.6, U14.25; no longer R51.6, U14.26
- net N$73: now also R26.7, U14.24; no longer R51.7, U14.27
- net N$74: now also R27.8, U14.27; no longer R51.8, U14.24
- net N$75: now also R26.5, U14.26; no longer R50.5, U14.25
- net N$76: now also R27.7, U14.28; no longer R50.8, U14.23
- net N$8: now also C26.1; no longer C6.1
- net N$83: now also IC2.7, R58.4; no longer IC1.7, R56.4
- net N$84: now also IC2.8, R59.1; no longer IC1.8, R57.1
- net N$85: now also IC2.9, R59.2; no longer IC1.9, R57.2
- net N$86: now also IC2.10, R59.3; no longer IC1.10, R57.3
- net N$87: now also IC2.11, R59.4; no longer IC1.11, R57.4
- net N$88: now also IC2.13; no longer IC1.13
- net N$89: now also R60.1; no longer R59.1
- net N$9: now also R13.2, U6.1; no longer R4.2, U5.1
- net N$90: now also R60.2; no longer R59.2
- net N$91: now also R60.3; no longer R59.3
- net N$92: now also R60.4; no longer R59.4
- net N$93: now also R61.1; no longer R60.1
- net N$94: now also R61.2; no longer R60.2
- net N$95: now also R61.3; no longer R60.3
- net N$96: now also LED7.A@7, R60.8; no longer LED1.A@7, R59.8
- net N$97: now also LED7.B@6, R60.7; no longer LED1.B@6, R59.7
- net N$98: now also LED7.C@4, R60.6; no longer LED1.C@4, R59.6
- net N$99: now also LED7.D@2, R60.5; no longer LED1.D@2, R59.5
- net PWM_DOT1: now also R17.1, U2.13; no longer R9.1, U4.13
- net PWM_DOT2: now also R18.1, U2.15; no longer R8.1, U4.15
- net PWM_SEG1: now also R10.1, U2.6; no longer R1.1, U4.6
- net PWM_SEG2: now also R11.1, U2.7; no longer R2.1, U4.7
- net PWM_SEG3: now also R12.1, U2.8; no longer R3.1, U4.8
- net PWM_SEG4: now also R13.1, U2.9; no longer R4.1, U4.9
- net PWM_SEG5: now also R14.1, U2.10; no longer R5.1, U4.10
- net PWM_SEG6: now also R15.1, U2.11; no longer R6.1, U4.11
- net PWM_SEG7: now also R16.1, U2.12; no longer R7.1, U4.12
- net RS485+: now also K5.A2, K5.B1, U17.6; no longer K3.A2, K3.B1, U15.6
- net RS485-: now also K5.A1, K5.B2, U17.7; no longer K3.A1, K3.B2, U15.7
- net RTC_1HZ_CLK: now also IC1.11, U1.7; no longer IC2.11, U13.7
- net SCK: now also IC1.3, K6.3, R23.2, R25.2, R27.2; no longer IC2.3, K17.3, R51.4, R52.4, R69.4
- net TCK: now also IC1.21, K7.1; no longer IC2.21, K18.1
- net TDI: now also IC1.24, K7.9; no longer IC2.24, K18.9
- net TDO: now also IC1.23, K7.3; no longer IC2.23, K18.3
- net TMS: now also IC1.22, K7.5; no longer IC2.22, K18.5
- net UART_DE: now also IC1.32, U17.3; no longer IC2.32, U15.3
- net UART_RX: now also R4.1, U17.1; no longer Q10.1, R18.1
- net UART_TX: now also IC1.10, U16.1, U17.4; no longer IC2.10, Q11.1, U15.4
- net VO: now also U3.5; no longer U1.5
- net VO1: now also U4.5; no longer U2.5
- net VO2: now also U5.5; no longer U3.5
- net VO3: now also U6.5; no longer U5.5
- net VO4: now also U7.5; no longer U6.5
- net VO5: now also U8.5; no longer U7.5
- net VO6: now also U9.5; no longer U8.5
- net VO7: now also Q9.G4, U11.5; no longer Q8.G4, U9.5
- net VO8: now also Q8.G4; no longer Q9.G4
- net X1: now also U1.1, Y2.P$1; no longer U13.1, X1.P$1
Routing:
- net AD1_BIASP: track 0.00 -> 47.6 mm
- net AD1_IEXC1: track 0.00 -> 24.4 mm
- net AD1_AIN1: track 0.00 -> 23.5 mm, vias 0 -> 2
- net AD1_AIN2: track 0.00 -> 22.0 mm, vias 0 -> 2
- net AD1_AIN3: track 0.00 -> 18.6 mm
- net AD1_AIN0: track 0.00 -> 17.3 mm
- net AD1_AIN6: track 0.00 -> 17.0 mm, vias 0 -> 2
- net AD1_AIN7: track 0.00 -> 15.2 mm
- net AD1_AIN5: track 0.00 -> 13.3 mm
- net AD1_AIN4: track 0.00 -> 11.5 mm
- net AD1_REFP0: track 0.00 -> 8.61 mm
- net AD1_REFN0: track 0.00 -> 8.42 mm
- net DVDD: track 0.00 -> 5.88 mm
- net N$30: track 0.00 -> 5.25 mm
- net N$51: track 0.00 -> 4.67 mm
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Other:
- board size 174.5 x 175 mm -> 175 x 175 mm

Commit message: small repositioning
Parts:
- moved C54 0.50 mm to (16.0, 9.00)
- moved C55 0.50 mm to (27.0, 9.00)
- moved C56 0.50 mm to (38.0, 9.00)
- moved C57 0.50 mm to (9.50, 9.00)
- moved C58 0.50 mm to (20.5, 9.00)
- moved C59 0.50 mm to (31.5, 9.00)
Routing:
- net AD1_AIN3: track 18.6 -> 19.6 mm
- net AD1_AIN1: track 23.5 -> 24.0 mm
- net AD1_AIN5: track 13.3 -> 13.8 mm
- net AD1_AIN7: track 15.2 -> 15.7 mm
- net AD1_AIN2: track 22.0 -> 22.5 mm
