File: SegmentDriver/SegmentDriver.brd (EAGLE design)
At the start: 175 x 175 mm, 244 parts, among them IC1 ATMEGA644A, IC2 PCA9555PW, IC3 4511D, K1 691313710002, K10 M02-MOLEX-104188-0210, K11 M02-MOLEX-104188-0210, K12 M02-MOLEX-104188-0210, K13 M02-MOLEX-104188-0210, K14 M02-MOLEX-104188-0210, K15 M02-MOLEX-104188-0210, K16 M02-MOLEX-104188-0210, K17 691210910004, K18 691210910004, K19 691210910004, K2 691313710002, K20 691210910004, K21 691210910004, K22 691210910004, K23 691210910004, K24 691210910004, K25 691210910004, K3 691322310002, K4 691322310002, K6 61200621621, K7 61201021621, K8 M02-MOLEX-104188-0210, K9 M02-MOLEX-104188-0210, Q1 MOSFET-NCHANNEL-FDMS5672, Q2 MOSFET-NCHANNEL-FDMS5672, Q3 MOSFET-NCHANNEL-FDMS5672, Q4 MOSFET-NCHANNEL-FDMS5672, Q5 MOSFET-NCHANNEL-FDMS5672, Q6 MOSFET-NCHANNEL-FDMS5672, Q7 MOSFET-NCHANNEL-FDMS5672, Q8 MOSFET-NCHANNEL-FDMS5672, Q9 MOSFET-NCHANNEL-FDMS5672, U1 DS1307SO8-TIGHT, U10 FOD8321, U11 FOD8321, U15 DMP2215L-7, U16 DMP2215L-7, U18 7808, U19 ADP3333ARM-5, U20 7805, U3 FOD8321, U4 FOD8321, U5 FOD8321, U6 FOD8321, U7 FOD8321, U8 FOD8321, U9 FOD8321, X1 53261-03, X2 53261-03, X3 53261-03, X4 53261-03, X5 53261-03, X6 53261-03, Y2 32.768kHz

Commit message: schematics finished (probably)
Parts:
- added C86, C87, C88, C89, C90, C91: 1uF, rcl:C0603K
- added R76, R77: 120, rcl:R0603
- added R78, R80, R82, R84, R86, R88: 69k, rcl:R0603
- added R79, R81, R83, R85, R87, R89: 18k, rcl:R0603
- added SW1, SW3, SW4, SW5, SW6, SW7: (no value), simbits:434153017835
- moved R75 164.8 mm to (74.0, -20.0), turned to 90 degrees
- moved R74 157.8 mm to (69.0, -20.0), turned to 90 degrees
- moved R73 150.9 mm to (64.0, -20.0), turned to 90 degrees
- moved R72 144.0 mm to (59.0, -20.0), turned to 90 degrees
- moved R71 137.1 mm to (54.0, -20.0), turned to 90 degrees
- moved LED1 129.0 mm to (32.5, 80.8)
- moved LED2 118.6 mm to (34.5, 70.0)
- moved U10 45.1 mm to (21.0, 124.5), turned to 90 degrees
- moved U11 36.2 mm to (39.0, 124.5), turned to 90 degrees
- moved LED6 35.2 mm to (151.5, 38.8)
- moved LED5 31.5 mm to (149.0, 39.5)
- moved LED3 15.9 mm to (10.0, 90.0)
- moved Q1 4.61 mm to (162.5, 131.0), turned to 0 degrees
- moved Q2 4.61 mm to (144.5, 131.0), turned to 0 degrees
- moved Q3 4.61 mm to (126.5, 131.0), turned to 0 degrees
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Connections:
- new net GPIO6_OUT: K5.B4, R76.2
- new net GPIO7_OUT: K5.B7, R77.2
- new net N$64: R78.2, R79.2, SW1.1, SW1.3, X1.2
- new net N$66: R80.2, R81.2, SW3.1, SW3.3, X2.2
- new net N$68: R82.2, R83.2, SW4.1, SW4.3, X3.2
- new net N$70: R84.2, R85.2, SW5.1, SW5.3, X4.2
- new net N$72: R86.2, R87.2, SW6.1, SW6.3, X5.2
- new net N$79: R88.2, R89.2, SW7.1, SW7.3, X6.2
- net +5V: now also R78.1, R80.1, R82.1, R84.1, R86.1, R88.1
- net AGND: now also C1.2, C3.2, C5.1, K1.2, K2.1, LED1.C, U10.4, U11.4, U3.4, U4.4, U5.4, U6.4, U7.4, U8.4, U9.4
- net GND: now also C86.1, C87.1, C88.1, C89.1, C90.1, C91.1, SW1.2, SW1.4, SW3.2, SW3.4, SW4.2, SW4.4, SW5.2, SW5.4, SW6.2, SW6.4, SW7.2, SW7.4; no longer C1.2, C3.2, C5.1, K1.2, K2.1, LED1.C, U10.4, U11.4, U3.4, U4.4, U5.4, U6.4, U7.4, U8.4, U9.4
- net GPIO0.0: now also C86.2, R79.1; no longer X1.2
- net GPIO0.1: now also C87.2, R81.1; no longer X2.2
- net GPIO0.2: now also C88.2, R83.1; no longer X3.2
- net GPIO0.3: now also C89.2, R85.1; no longer X4.2
- net GPIO0.4: now also C90.2, R87.1; no longer X5.2
- net GPIO0.5: now also C91.2, R89.1; no longer X6.2
- net GPIO0.6_OUT: now also R76.1; no longer K5.B4
- net GPIO0.7_OUT: now also R77.1; no longer K5.B7
Routing:
- net +15V: track 30.6 -> 104.1 mm
- net VO: track 58.2 -> 0.00 mm
- net VO8: track 54.1 -> 0.00 mm
- net VO1: track 48.2 -> 0.00 mm
- net VO7: track 44.2 -> 0.00 mm
- net VO2: track 37.2 -> 0.00 mm
- net VO6: track 34.4 -> 0.00 mm
- net VO3: track 28.6 -> 0.00 mm
- net GND: track 58.8 -> 32.6 mm
- net VO5: track 22.2 -> 0.00 mm
- net VO4: track 19.3 -> 0.00 mm
- net N$66: track 0.00 -> 8.99 mm, vias 0 -> 1
- net N$64: track 0.00 -> 8.99 mm, vias 0 -> 1
- net N$79: track 0.00 -> 8.99 mm, vias 0 -> 1
- net N$72: track 0.00 -> 8.99 mm, vias 0 -> 1
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- added copper zone on layer 1, net +24V
- added copper zone on layer 16, net +24V
- added copper zone on layer 1, net AGND
- added copper zone on layer 1, net N$11
- added copper zone on layer 1, net N$13
- added copper zone on layer 1, net N$15
- added copper zone on layer 1, net N$17
- added copper zone on layer 1, net N$18
- added copper zone on layer 1, net N$19
- added copper zone on layer 1, net N$3
- added copper zone on layer 1, net N$6
- added copper zone on layer 1, net N$8
