File: SegmentDriver/SegmentDriver_no_heaters.brd (EAGLE design)
At the start: 175 x 175 mm, 270 parts, among them IC1 ATMEGA644A, IC2 PCA9555PW, IC3 4511D, K1 691313710002, K10 M02-MOLEX-104188-0210, K11 M02-MOLEX-104188-0210, K12 M02-MOLEX-104188-0210, K13 M02-MOLEX-104188-0210, K14 M02-MOLEX-104188-0210, K15 M02-MOLEX-104188-0210, K16 M02-MOLEX-104188-0210, K17 691210910004, K18 691210910004, K19 691210910004, K2 691313710002, K20 691210910004, K21 691210910004, K22 691210910004, K23 691210910004, K24 691210910004, K25 691210910004, K3 691322310002, K4 691322310002, K6 61200621621, K7 61201021621, K8 M02-MOLEX-104188-0210, K9 M02-MOLEX-104188-0210, Q1 MOSFET-NCHANNEL-FDMS5672, Q2 MOSFET-NCHANNEL-FDMS5672, Q3 MOSFET-NCHANNEL-FDMS5672, Q4 MOSFET-NCHANNEL-FDMS5672, Q5 MOSFET-NCHANNEL-FDMS5672, Q6 MOSFET-NCHANNEL-FDMS5672, Q7 MOSFET-NCHANNEL-FDMS5672, Q8 MOSFET-NCHANNEL-FDMS5672, Q9 MOSFET-NCHANNEL-FDMS5672, U1 DS1307SO8-TIGHT, U10 FOD8321, U11 FOD8321, U15 DMP2215L-7, U16 DMP2215L-7, U18 7808, U19 ADP3333ARM-5, U20 7805, U3 FOD8321, U4 FOD8321, U5 FOD8321, U6 FOD8321, U7 FOD8321, U8 FOD8321, U9 FOD8321, X1 53261-03, X2 53261-03, X3 53261-03, X4 53261-03, X5 53261-03, X6 53261-03, Y2 32.768kHz

Commit message: Seperation of heaters and drivers
Parts:
- removed C1, C3: 220UF, Panasonic-EEEFK_EEEFP:CAPAE1900X1700N
- removed C15, C16, C17, C18, C19, C20, C21, C22, C23: 0.1uF, rcl:C1206K
- removed C24, C25, C26, C27, C28, C29, C30, C31, C32: 100UF, Panasonic-EEEFK_EEEFP:CAPAE1700X1700N
- removed C5: 0.1uF, rcl:C0603K
- removed K1, K2: 691313710002, Wurth_Elektronik_Electromechanic_Terminal_Blocks_Connectors_rev15d:691313710002
- removed K10, K11, K12, K13, K14, K15, K16, K8, K9: M02-MOLEX-104188-0210, simbits:LITE-TRAP-CONNECTOR-2
- removed LED1: (no value), adafruit:CHIPLED_0603
- removed Q1, Q2, Q3, Q4, Q5, Q6, Q7, Q8, Q9: MOSFET-NCHANNEL-FDMS5672, simbits:POWERPACK5060-8
- removed R1: 2K4, rcl:R0603
- removed R10, R11, R12, R13, R14, R15, R16, R17, R18: 330, rcl:R0603
- removed U10, U11, U3, U4, U5, U6, U7, U8, U9: FOD8321, simbits:WB-SOP5
Connections:
- removed net +24V: C1.1, C3.1, C5.2, K1.1, K10.2A, K10.2B, K11.2A, K11.2B, K12.2A, K12.2B, K13.2A, K13.2B, K14.2A, K14.2B, K15.2A, K15.2B, K16.2A, K16.2B, K2.2, K8.2A, K8.2B, K9.2A, K9.2B, R1.2
- removed net AGND: C1.2, C24.2, C25.2, C26.2, C27.2, C28.2, C29.2, C3.2, C30.2, C31.2, C32.2, C5.1, K1.2, K2.1, LED1.C, Q1.S1, Q1.S2, Q1.S3, Q2.S1, Q2.S2, Q2.S3, Q3.S1, Q3.S2, Q3.S3, Q4.S1, Q4.S2, Q4.S3, Q5.S1, Q5.S2, Q5.S3, Q6.S1, Q6.S2, Q6.S3, Q7.S1, Q7.S2, Q7.S3, Q8.S1, Q8.S2, Q8.S3, Q9.S1, Q9.S2, Q9.S3, U10.4, U11.4, U3.4, U4.4, U5.4, U6.4, U7.4, U8.4, U9.4
- removed net N$1: R18.2, U11.1
- removed net N$10: R10.2, U3.1
- removed net N$11: C27.1, K11.1A, K11.1B, Q4.D5, Q4.D6, Q4.D7, Q4.D8, Q4.DPAD
- removed net N$12: R14.2, U7.1
- removed net N$13: C28.1, K12.1A, K12.1B, Q5.D5, Q5.D6, Q5.D7, Q5.D8, Q5.DPAD
- removed net N$14: R15.2, U8.1
- removed net N$15: C29.1, K13.1A, K13.1B, Q6.D5, Q6.D6, Q6.D7, Q6.D8, Q6.DPAD
- removed net N$16: R16.2, U9.1
- removed net N$17: C30.1, K14.1A, K14.1B, Q7.D5, Q7.D6, Q7.D7, Q7.D8, Q7.DPAD
- removed net N$18: C31.1, K15.1A, K15.1B, Q8.D5, Q8.D6, Q8.D7, Q8.D8, Q8.DPAD
- removed net N$19: C32.1, K16.1A, K16.1B, Q9.D5, Q9.D6, Q9.D7, Q9.D8, Q9.DPAD
- removed net N$2: R17.2, U10.1
- removed net N$3: C24.1, K8.1A, K8.1B, Q1.D5, Q1.D6, Q1.D7, Q1.D8, Q1.DPAD
- removed net N$4: R11.2, U4.1
- removed net N$6: C25.1, K9.1A, K9.1B, Q2.D5, Q2.D6, Q2.D7, Q2.D8, Q2.DPAD
- removed net N$63: LED1.A, R1.1
- removed net N$7: R12.2, U5.1
- removed net N$8: C26.1, K10.1A, K10.1B, Q3.D5, Q3.D6, Q3.D7, Q3.D8, Q3.DPAD
- removed net N$9: R13.2, U6.1
- removed net PWM_DOT1: R17.1, U2.13
- removed net PWM_DOT2: R18.1, U2.15
- removed net VO: Q1.G4, U3.5
- removed net VO1: Q2.G4, U4.5
- removed net VO2: Q3.G4, U5.5
- removed net VO3: Q4.G4, U6.5
- removed net VO4: Q5.G4, U7.5
- removed net VO5: Q6.G4, U8.5
- removed net VO6: Q7.G4, U9.5
- removed net VO7: Q9.G4, U11.5
- removed net VO8: Q8.G4, U10.5
- new net PWM_SEG10: U2.16
- new net PWM_SEG11: U2.17
- new net PWM_SEG12: U2.18
- new net PWM_SEG13: U2.19
- new net PWM_SEG14: U2.20
- new net PWM_SEG15: U2.21
- new net PWM_SEG16: U2.22
- new net PWM_SEG8: U2.13
- new net PWM_SEG9: U2.15
- net +15V: no longer C15.1, C16.1, C17.1, C18.1, C19.1, C20.1, C21.1, C22.1, C23.1, U10.6, U11.6, U3.6, U4.6, U5.6, U6.6, U7.6, U8.6, U9.6
- net GND: no longer C15.2, C16.2, C17.2, C18.2, C19.2, C20.2, C21.2, C22.2, C23.2, U10.3, U11.3, U3.3, U4.3, U5.3, U6.3, U7.3, U8.3, U9.3
- net PWM_SEG1: no longer R10.1
- net PWM_SEG2: no longer R11.1
- net PWM_SEG3: no longer R12.1
- net PWM_SEG4: no longer R13.1
- net PWM_SEG5: no longer R14.1
- net PWM_SEG6: no longer R15.1
- net PWM_SEG7: no longer R16.1
Routing:
- net +15V: track 104.1 -> 0.00 mm
- net GND: track 32.6 -> 29.6 mm
- removed copper zone on layer 1, net +24V
- removed copper zone on layer 16, net +24V
- removed copper zone on layer 1, net AGND
- removed copper zone on layer 1, net N$11
- removed copper zone on layer 1, net N$13
- removed copper zone on layer 1, net N$15
- removed copper zone on layer 1, net N$17
- removed copper zone on layer 1, net N$18
- removed copper zone on layer 1, net N$19
- removed copper zone on layer 1, net N$3
- removed copper zone on layer 1, net N$6
- removed copper zone on layer 1, net N$8
