File: SegmentDriver/SegmentDriver_no_heaters.sch (EAGLE design)
At the start: 269 parts, among them IC1 ATMEGA644A, IC2 PCA9555PW, IC3 4511D, K1 691313710002, K10 M02-MOLEX-104188-0210, K11 M02-MOLEX-104188-0210, K12 M02-MOLEX-104188-0210, K13 M02-MOLEX-104188-0210, K14 M02-MOLEX-104188-0210, K15 M02-MOLEX-104188-0210, K16 M02-MOLEX-104188-0210, K17 691210910004, K18 691210910004, K19 691210910004, K2 691313710002, K20 691210910004, K21 691210910004, K22 691210910004, K23 691210910004, K24 691210910004, K25 691210910004, K3 691322310002, K4 691322310002, K6 61200621621, K7 61201021621, K8 M02-MOLEX-104188-0210, K9 M02-MOLEX-104188-0210, Q1 MOSFET-NCHANNEL-FDMS5672, Q2 MOSFET-NCHANNEL-FDMS5672, Q3 MOSFET-NCHANNEL-FDMS5672, Q4 MOSFET-NCHANNEL-FDMS5672, Q5 MOSFET-NCHANNEL-FDMS5672, Q6 MOSFET-NCHANNEL-FDMS5672, Q7 MOSFET-NCHANNEL-FDMS5672, Q8 MOSFET-NCHANNEL-FDMS5672, Q9 MOSFET-NCHANNEL-FDMS5672, U1 DS1307SO8-TIGHT, U10 FOD8321, U11 FOD8321, U15 DMP2215L-7, U16 DMP2215L-7, U18 7808, U19 ADP3333ARM-5, U20 7805, U3 FOD8321, U4 FOD8321, U5 FOD8321, U6 FOD8321, U7 FOD8321, U8 FOD8321, U9 FOD8321, X1 53261-03, X2 53261-03, X3 53261-03, X4 53261-03, X5 53261-03, X6 53261-03, Y2 32.768kHz

Commit message: Seperation of heaters and drivers
Parts:
- removed C1, C3: 220UF, Panasonic-EEEFK_EEEFP:EEE-FK2A221AM-CASE-K16
- removed C15, C16, C17, C18, C19, C20, C21, C22, C23: 0.1uF, rcl:C-EUC1206K
- removed C24, C25, C26, C27, C28, C29, C30, C31, C32: 100UF, Panasonic-EEEFK_EEEFP:EEE-FK2A101AM-CASE-J16
- removed C5: 0.1uF, rcl:C-EUC0603K
- removed K1, K2: 691313710002, Wurth_Elektronik_Electromechanic_Terminal_Blocks_Connectors_rev15d:691313710002
- removed K10, K11, K12, K13, K14, K15, K16, K8, K9: M02-MOLEX-104188-0210, simbits:M02-MOLEX-104188-0210
- removed LED1: (no value), adafruit:LEDCHIPLED_0603
- removed Q1, Q2, Q3, Q4, Q5, Q6, Q7, Q8, Q9: MOSFET-NCHANNEL-FDMS5672, simbits:MOSFET-NCHANNEL-FDMS5672
- removed R1: 2K4, rcl:R-EU_R0603
- removed R10, R11, R12, R13, R14, R15, R16, R17, R18: 330, rcl:R-EU_R0603
- removed U10, U11, U3, U4, U5, U6, U7, U8, U9: FOD8321, simbits:FOD8321
Connections:
- removed net +24V: C1.1, C3.1, C5.2, K1.1, K10.2, K11.2, K12.2, K13.2, K14.2, K15.2, K16.2, K2.2, K8.2, K9.2, R1.2
- removed net AGND: C1.2, C24.2, C25.2, C26.2, C27.2, C28.2, C29.2, C3.2, C30.2, C31.2, C32.2, C5.1, K1.2, K2.1, LED1.C, Q1.S, Q2.S, Q3.S, Q4.S, Q5.S, Q6.S, Q7.S, Q8.S, Q9.S, U10.VSS@4, U11.VSS@4, U3.VSS@4, U4.VSS@4, U5.VSS@4, U6.VSS@4, U7.VSS@4, U8.VSS@4, U9.VSS@4
- removed net N$1: R18.2, U11.A@1
- removed net N$10: R10.2, U3.A@1
- removed net N$11: C27.1, K11.1, Q4.D
- removed net N$12: R14.2, U7.A@1
- removed net N$13: C28.1, K12.1, Q5.D
- removed net N$14: R15.2, U8.A@1
- removed net N$15: C29.1, K13.1, Q6.D
- removed net N$16: R16.2, U9.A@1
- removed net N$17: C30.1, K14.1, Q7.D
- removed net N$18: C31.1, K15.1, Q8.D
- removed net N$19: C32.1, K16.1, Q9.D
- removed net N$2: R17.2, U10.A@1
- removed net N$3: C24.1, K8.1, Q1.D
- removed net N$4: R11.2, U4.A@1
- removed net N$6: C25.1, K9.1, Q2.D
- removed net N$63: LED1.A, R1.1
- removed net N$7: R12.2, U5.A@1
- removed net N$8: C26.1, K10.1, Q3.D
- removed net N$9: R13.2, U6.A@1
- removed net PWM_DOT1: R17.1, U2.PWM7
- removed net PWM_DOT2: R18.1, U2.PWM8
- removed net VO: Q1.G, U3.VO@5
- removed net VO1: Q2.G, U4.VO@5
- removed net VO2: Q3.G, U5.VO@5
- removed net VO3: Q4.G, U6.VO@5
- removed net VO4: Q5.G, U7.VO@5
- removed net VO5: Q6.G, U8.VO@5
- removed net VO6: Q7.G, U9.VO@5
- removed net VO7: Q9.G, U11.VO@5
- removed net VO8: Q8.G, U10.VO@5
- new net PWM_SEG10: U2.PWM9
- new net PWM_SEG11: U2.PWM10
- new net PWM_SEG12: U2.PWM11
- new net PWM_SEG13: U2.PWM12
- new net PWM_SEG14: U2.PWM13
- new net PWM_SEG15: U2.PWM14
- new net PWM_SEG16: U2.PWM15
- new net PWM_SEG8: U2.PWM7
- new net PWM_SEG9: U2.PWM8
- net +15V: no longer C15.1, C16.1, C17.1, C18.1, C19.1, C20.1, C21.1, C22.1, C23.1, U10.VDD@6, U11.VDD@6, U3.VDD@6, U4.VDD@6, U5.VDD@6, U6.VDD@6, U7.VDD@6, U8.VDD@6, U9.VDD@6
- net GND: no longer C15.2, C16.2, C17.2, C18.2, C19.2, C20.2, C21.2, C22.2, C23.2, U10.K@3, U11.K@3, U3.K@3, U4.K@3, U5.K@3, U6.K@3, U7.K@3, U8.K@3, U9.K@3
- net PWM_SEG1: no longer R10.1
- net PWM_SEG2: no longer R11.1
- net PWM_SEG3: no longer R12.1
- net PWM_SEG4: no longer R13.1
- net PWM_SEG5: no longer R14.1
- net PWM_SEG6: no longer R15.1
- net PWM_SEG7: no longer R16.1
Other:
- note removed: "Heater output stage"
- note removed: "PWR 24V"
